File: hardware/0.2-ext/sea-picro.kicad_pcb (KiCad board)
At the start: 4 copper layers, 17.8 x 33 mm, 59 parts, among them J1 USB_C_Receptacle_USB2.0, J2 0.1" x 12, J3 0.1" x 12, J4 D+, J5 D-, J6 0.1" x 5, J7 2.54, Q1 2N7002VC-7, Q2 2N7002VC-7, U1 AP7365-33WG-7, U2 GD25Q64CWIGR, U3 RP2040, U4 74LVC1T45Z6-7, Y1 12MHz

Commit message: Fix IO 12 silk in EXT
Other:
- board text added: "12"
- board text removed: "15"
Changed lines of the file:
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@@
     (effects (font (size 1 1) (thickness 0.15)) (justify mirror))
   )
-  (gr_text "15" (at 126.2 104.7 90) (layer "B.SilkS")
+  (gr_text "12" (at 126.2 104.7 90) (layer "B.SilkS")
     (effects (font (size 1 1) (thickness 0.15)) (justify mirror))
   )
