File: hardware/0.3-ext/sea-picro.kicad_pcb (KiCad board)
At the start: 4 copper layers, 17.8 x 33 mm, 59 parts, among them J1 USB_C_Receptacle_USB2.0, J2 0.1" x 12, J3 0.1" x 12, J4 D+, J5 D-, J6 0.1" x 5, J7 2.54, Q1 2N7002VC-7, Q2 2N7002VC-7, U1 AP7365-33WG-7, U2 GD25Q64CWIGR, U3 RP2040, U4 74LVC1T45Z6-7, Y1 12MHz

Commit message: Remove Pin 12 message
Other:
- board text removed: "PIN 12 LABELED INCORRECTLY ON BACK SILK"
Changed lines of the file:
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@@
-    (effects (font (size 1 1) (thickness 0.15)))
-  )
-  (gr_text "PIN 12 LABELED\nINCORRECTLY ON \nBACK SILK" (at 126.3 110.9) (layer "Dwgs.User")
     (effects (font (size 1 1) (thickness 0.15)))
   )

Commit message: clean up routing
Parts:
- moved LOGO1 0.20 mm to (126.2, 99.8)
Routing:
- net /nRST: track 9.38 -> 14.9 mm
- net /15: track 11.0 -> 8.70 mm
- net /SWDIO: track 6.08 -> 7.63 mm
- net /VBUS_DETECT: track 23.1 -> 22.1 mm
- net /12: track 11.8 -> 11.0 mm
