File: hardware/0.3-rst/sea-picro.kicad_pcb (KiCad board)
At the start: 4 copper layers, 17.8 x 33 mm, 59 parts, among them J1 USB_C_Receptacle_USB2.0, J2 0.1" x 12, J3 0.1" x 12, J4 D+, J5 D-, Q1 2N7002VC-7, Q2 2N7002VC-7, SW1 SWITCH, U1 AP7365-33WG-7, U2 GD25Q64CWIGR, U3 RP2040, Y1 12MHz

Commit message: clean up routing
Parts:
- removed TP2: DELAY, josh-test-point:TestPoint_SMDPad_D1.0mm_NO_SILK
- moved LOGO1 0.10 mm to (126.2, 99.7)
Routing:
- net /VBUS_DETECT: track 24.7 -> 19.4 mm, vias 2 -> 3
- net Net-(C19-Pad1): track 10.0 -> 7.98 mm, vias 1 -> 0
- net /SWDIO: track 8.13 -> 6.75 mm
Other:
- board text removed: "DEL"
