File: hardware/0.3-ext-castellated-melted/sea-picro.kicad_sch (KiCad schematic)
At the start: 54 parts, among them J1 USB_C_Receptacle_USB2.0, J2 Sea-Picro, Q1 2N7002VC-7, Q2 2N7002VC-7, U1 XC6210B332MR-G, U2 GD25Q64CWIGR, U3 RP2040, U4 74LVC1T45, Y1 12MHz

Commit message: fix 1u cap bom
Parts:
- C12, C9: LCSC C15849 -> C52923; MPN  CL10A105KB8NNNC -> CL05A105KA5NQNC
Changed lines of the file:
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@@
       (effects (font (size 1.27 1.27)) hide)
     )
-    (property "LCSC" "C15849" (id 4) (at 131.445 74.93 0)
-      (effects (font (size 1.27 1.27)) hide)
-    )
-    (property "MPN " "CL10A105KB8NNNC" (id 5) (at 131.445 74.93 0)
+    (property "LCSC" "C52923" (id 4) (at 131.445 74.93 0)
+      (effects (font (size 1.27 1.27)) hide)
+    )
+    (property "MPN " "CL05A105KA5NQNC" (id 5) (at 131.445 74.93 0)
       (effects (font (size 1.27 1.27)) hide)
     )
@@
       (effects (font (size 1.27 1.27)) hide)
     )
-    (property "LCSC" "C15849" (id 4) (at 138.43 60.96 0)
-      (effects (font (size 1.27 1.27)) hide)
-    )
-    (property "MPN " "CL10A105KB8NNNC" (id 5) (at 138.43 60.96 0)
-      (effects (font (size 1.27 1.27)) hide)
-    )
+    (property "LCSC" "C52923" (id 4) (at 138.43 60.96 0)
+      (effects (font (size 1.27 1.27)) hide)
+    )
+    (property "MPN " "CL05A105KA5NQNC" (id 5) (at 138.43 60.96 0)
+      (effects (font (size 1.27 1.27)) hide)
+    )
